File: PCB/Combine/Dock/DeviceSelect.kicad_sch (KiCad schematic)
At the start: 30 parts, among them U4 SIP32509DT-T1-GE3, U5 USB2422T-I/MJ, U6 SIP32509DT-T1-GE3, Y1 X322524MOB4SI

Commit message: Adding some renders
Other:
- company: (none) -> DK
- title: (none) -> BLEarrings V1
