File: PCB/Combine/Dock/Dock.kicad_sch (KiCad schematic)
At the start: 16 parts, among them J1 Conn_01x10_Socket, J1 USB_C_Receptacle, P1 USB_C_Plug, P2 USB_C_Plug

Commit message: Adding some renders
Other:
- company: (none) -> DK
- title: (none) -> BLEarrings V1
