File: PCB/Combine/Dock/DockBattery.kicad_sch (KiCad schematic)
At the start: 28 parts, among them U1 AMS1117-3.3, U2 BQ24073RGT, U3 TPS61023DRLR

Commit message: Adding some renders
Other:
- company: (none) -> DK
- title: (none) -> BLEarrings V1
