File: PCB/Combine/EarringLeft/BLEEarrings.kicad_sch (KiCad schematic)
At the start: 5 parts, among them J6 USB_C_Receptacle, SW3 TK-6580B-1

Commit message: Adding some renders
Other:
- company: Kitty and Dom -> DK
- title: BLEEarrings (Blade Runner) -> BLEarrings V1
