File: PCB/Combine/EarringLeft/DSP.kicad_sch (KiCad schematic)
At the start: 39 parts, among them J7 Screw_Terminal_01x01, J8 Screw_Terminal_01x02, SW4 SW_DIP_x01, U10 NRF52833-QDAA-R7, Y4 X161032768KLD2SI, Y5 XL7EL89CKI-111YLC-32M

Commit message: Adding some renders
Parts:
- Y4: value X161032768KLD2SI -> X161032768KLD2SI
- Y5: value XL7EL89CKI-111YLC-32M -> XL7EL89CKI-111YLC-32M
Other:
- company: Kitty and Dom -> DK
- title: BLEEarrings (Blade Runner) -> BLEarrings V1
