File: PCB/Combine/EarringLeft/Power.kicad_sch (KiCad schematic)
At the start: 10 parts, among them U11 MCP73831T-2ACI/OT, U12 XB6096I2SV

Commit message: Adding some renders
Other:
- company: Kitty and Dom -> DK
- title: BLEEarrings (Blade Runner) -> BLEarrings V1
