File: PCB/Combine/EarringRight/BLEEarrings.kicad_sch (KiCad schematic)
At the start: 5 parts, among them J3 USB_C_Receptacle, SW1 TK-6580B-1

Commit message: Adding some renders
Other:
- company: Kitty and Dom -> DK
- title: BLEEarrings (Blade Runner) -> BLEarrings V1
