File: PCB/Combine/EarringRight/DSP.kicad_sch (KiCad schematic)
At the start: 40 parts, among them J4 Screw_Terminal_01x01, J5 Screw_Terminal_01x02, SW2 SW_DIP_x01, U9 NRF52833-QDAA-R7, Y2 X161032768KLD2SI, Y3 XL7EL89CKI-111YLC-32M

Commit message: Adding some renders
Parts:
- Y2: value X161032768KLD2SI -> X161032768KLD2SI
- Y3: value XL7EL89CKI-111YLC-32M -> XL7EL89CKI-111YLC-32M
Other:
- company: Kitty and Dom -> DK
- title: BLEEarrings (Blade Runner) -> BLEarrings V1
